Commit message: new test

File: urdf_generator/mypackage/robot.urdf (robot description, URDF)
Before this commit: robot gummi, 7 links, 6 joints
Links:
- removed link link2
- removed link link4
- removed link link5
- removed link link6
Joints:
- removed joint joint10
- removed joint joint11
- removed joint joint12
- removed joint joint7
- removed joint joint8
- removed joint joint9
- added joint joint2: type continuous, parent base_link, child link1, origin xyz=3.552713678800501e-17 -2.3665827156630353e-32 -4.440892098500626e-18 rpy=0 0 0, axis 0.0 1.0 0.0, limit lower=-1 upper=1 effort=0 velocity=0
- added joint joint4: type continuous, parent link1, child link3, origin xyz=-1.7763568394002506e-16 0.12800000000000034 -2.486899575160351e-16 rpy=0 0 0, axis -3.400058012914542e-16 -1.0475804435582063e-16 -1.0000000000000004, limit lower=-1 upper=1 effort=0 velocity=0

Commit message: newest test

File: urdf_generator/mypackage/robot.urdf (robot description, URDF)
Before this commit: robot gummi, 3 links, 2 joints
Links:
- added link base, mass 0; collision mesh filename=package://mypackage/meshes/base.stl; visual mesh filename=package://mypackage/meshes/base.stl
- added link link2, mass 0; collision mesh filename=package://mypackage/meshes/link2.stl; visual mesh filename=package://mypackage/meshes/link2.stl
- added link link4, mass 0; collision mesh filename=package://mypackage/meshes/link4.stl; visual mesh filename=package://mypackage/meshes/link4.stl
- added link link5, mass 0; collision mesh filename=package://mypackage/meshes/link5.stl; visual mesh filename=package://mypackage/meshes/link5.stl
- link base_link: mass 0 -> None; geometry 
Joints:
- removed joint joint2
- removed joint joint4
- added joint joint10: type continuous, parent link4, child link5, origin xyz=-0.030000000000000887 -0.173499999999998 -0.13400000000000076 rpy=0 0 0, axis 1.0000000000000009 8.062965342091539e-18 9.714451465470163e-17, limit lower=-1 upper=1 effort=0 velocity=0
- added joint joint6: type continuous, parent base, child link1, origin xyz=3.552713678800501e-17 -2.3665827156630353e-32 -4.440892098500626e-18 rpy=0 0 0, axis 0.0 1.0 0.0, limit lower=-1 upper=1 effort=0 velocity=0
- added joint joint7: type continuous, parent link1, child link2, origin xyz=-1.7763568394002506e-16 0.12800000000000034 -2.486899575160351e-16 rpy=0 0 0, axis -3.400058012914542e-16 -1.0475804435582063e-16 -1.0000000000000004, limit lower=-1 upper=1 effort=0 velocity=0
- added joint joint8: type continuous, parent link2, child link3, origin xyz=9.769962616701378e-17 0.12800000000000047 -0.13400000000000037 rpy=0 0 0, axis -0.9999999999999994 2.2204460492503116e-16 -3.677613769070831e-16, limit lower=-1 upper=1 effort=0 velocity=0
- added joint joint9: type continuous, parent link3, child link4, origin xyz=-0.030000000000000818 0.06450000000000117 -0.1340000000000005 rpy=0 0 0, axis -1.634803403760541e-14 -0.9999999999999962 1.0475804435583023e-16, limit lower=-1 upper=1 effort=0 velocity=0
- added joint set_worldaxis: type , parent base_link, child base, origin xyz=0 0 0 rpy=1.570796326795 0 0, axis 0 0 0, limit lower=-1 upper=1 effort=0 velocity=0

Commit message: new testo

File: urdf_generator/mypackage/robot.urdf (robot description, URDF)
Before this commit: robot gummi, 7 links, 6 joints
Links:
- removed link link2
- removed link link4
Joints:
- removed joint joint10
- removed joint joint7
- removed joint joint8
- removed joint joint9
- added joint joint2: type continuous, parent base, child link1, origin xyz=3.552713678800501e-17 -2.3665827156630353e-32 -4.440892098500626e-18 rpy=0 0 0, axis 0.0 1.0 0.0, limit lower=-1 upper=1 effort=0 velocity=0
- added joint joint4: type continuous, parent link1, child link3, origin xyz=-2.1316282072803005e-16 0.12800000000000034 -2.4424906541753446e-16 rpy=0 0 0, axis -3.400058012914542e-16 -1.0475804435582063e-16 -1.0000000000000004, limit lower=-1 upper=1 effort=0 velocity=0
- joint joint6: axis 0.0 1.0 0.0 -> -0.9999999999999994 2.2204460492503116e-16 -3.677613769070831e-16; child link1 -> link5; origin xyz=3.552713678800501e-17 -2.3665827156630353e-32 -4.440892098500626e-18 rpy=0 0 0 -> xyz=2.753353101070388e-16 1.4210854715202004e-16 -0.13400000000000012 rpy=0 0 0; parent base -> link3
- joint set_worldaxis: origin xyz=0 0 0 rpy=1.570796326795 0 0 -> xyz=0 0 0 rpy=0 0 0; type  -> fixed

Commit message: new testooo

File: urdf_generator/mypackage/robot.urdf (robot description, URDF)
Before this commit: robot gummi, 5 links, 4 joints
Links:
- added link link2, mass 0; collision mesh filename=package://mypackage/meshes/link2.stl; visual mesh filename=package://mypackage/meshes/link2.stl
- added link link4, mass 0; collision mesh filename=package://mypackage/meshes/link4.stl; visual mesh filename=package://mypackage/meshes/link4.stl
Joints:
- removed joint joint6
- added joint joint0: type continuous, parent base, child link1, origin xyz=3.552713678800501e-17 -2.3665827156630353e-32 -4.440892098500626e-18 rpy=0 0 0, axis 0.0 1.0 0.0, limit lower=-1 upper=1 effort=0 velocity=0
- added joint joint1: type continuous, parent link1, child link2, origin xyz=-2.1316282072803005e-16 0.12800000000000034 -2.4424906541753446e-16 rpy=0 0 0, axis -3.400058012914542e-16 -1.0475804435582063e-16 -1.0000000000000004, limit lower=-1 upper=1 effort=0 velocity=0
- added joint joint3: type continuous, parent link3, child link4, origin xyz=-0.030000000000000915 -0.06349999999999931 -1.5987211554602254e-16 rpy=0 0 0, axis -1.634803403760541e-14 -0.9999999999999962 1.0475804435583023e-16, limit lower=-1 upper=1 effort=0 velocity=0
- joint joint2: axis 0.0 1.0 0.0 -> -0.9999999999999994 2.2204460492503116e-16 -3.677613769070831e-16; child link1 -> link3; origin xyz=3.552713678800501e-17 -2.3665827156630353e-32 -4.440892098500626e-18 rpy=0 0 0 -> xyz=2.753353101070388e-16 1.4210854715202004e-16 -0.13400000000000012 rpy=0 0 0; parent base -> link2
- joint joint4: axis -3.400058012914542e-16 -1.0475804435582063e-16 -1.0000000000000004 -> 1.0000000000000009 8.062965342091539e-18 9.714451465470163e-17; child link3 -> link5; origin xyz=-2.1316282072803005e-16 0.12800000000000034 -2.4424906541753446e-16 rpy=0 0 0 -> xyz=-7.105427357601002e-17 -0.23799999999999916 -2.486899575160351e-16 rpy=0 0 0; parent link1 -> link4
- joint set_worldaxis: origin xyz=0 0 0 rpy=0 0 0 -> xyz=0 0 0 rpy=1.570796326795 0 0
